Commit message: feat: add go2-piper keyplay, clean URDF paths, and tune body/force-estimate kp-kd in go2 config

File: resources/robots/go2_piper/go2/urdf/go2_description.urdf (robot description, URDF)
Before this commit: robot go2_description, 29 links, 28 joints
Links:
- link FL_calf: geometry collision cylinder length=0.12 radius=0.012; visual mesh filename=../dae/calf.dae
- link FL_foot: geometry collision sphere radius=0.022; visual mesh filename=../dae/foot.dae
- link FL_hip: geometry collision cylinder length=0.04 radius=0.046; visual mesh filename=../dae/hip.dae
- link FL_thigh: geometry collision box size=0.213 0.0245 0.034; visual mesh filename=../dae/thigh.dae
- link FR_calf: geometry collision cylinder length=0.12 radius=0.013; visual mesh filename=../dae/calf_mirror.dae
- link FR_foot: geometry collision sphere radius=0.022; visual mesh filename=../dae/foot.dae
- link FR_hip: geometry collision cylinder length=0.04 radius=0.046; visual mesh filename=../dae/hip.dae
- link FR_thigh: geometry collision box size=0.213 0.0245 0.034; visual mesh filename=../dae/thigh_mirror.dae
- link RL_calf: geometry collision cylinder length=0.12 radius=0.013; visual mesh filename=../dae/calf.dae
- link RL_foot: geometry collision sphere radius=0.022; visual mesh filename=../dae/foot.dae
- link RL_hip: geometry collision cylinder length=0.04 radius=0.046; visual mesh filename=../dae/hip.dae
- link RL_thigh: geometry collision box size=0.213 0.0245 0.034; visual mesh filename=../dae/thigh.dae
- link RR_calf: geometry collision cylinder length=0.12 radius=0.013; visual mesh filename=../dae/calf_mirror.dae
- link RR_foot: geometry collision sphere radius=0.022; visual mesh filename=../dae/foot.dae
- link RR_hip: geometry collision cylinder length=0.04 radius=0.046; visual mesh filename=../dae/hip.dae
- link RR_thigh: geometry collision box size=0.213 0.0245 0.034; visual mesh filename=../dae/thigh_mirror.dae
- link base: geometry collision box size=0.3762 0.0935 0.114; visual mesh filename=../dae/base.dae

File: resources/robots/go2_piper/piper_description/urdf/piper_with_gripper.urdf (robot description, URDF)
Before this commit: robot piper, 12 links, 10 joints
Links:
- link base_link: geometry collision mesh filename=../meshes/base_link.STL; visual mesh filename=../meshes/base_link.STL
- link gripper_base: geometry collision mesh filename=../meshes/gripper_base.STL; visual mesh filename=../meshes/gripper_base.STL
- link link1: geometry collision mesh filename=../meshes/link1.STL; visual mesh filename=../meshes/link1.STL
- link link2: geometry collision mesh filename=../meshes/link2.STL; visual mesh filename=../meshes/link2.STL
- link link3: geometry collision mesh filename=../meshes/link3.STL; visual mesh filename=../meshes/link3.STL
- link link4: geometry collision mesh filename=../meshes/link4.STL; visual mesh filename=../meshes/link4.STL
- link link5: geometry collision mesh filename=../meshes/link5.STL; visual mesh filename=../meshes/link5.STL
- link link6: geometry collision mesh filename=../meshes/link6.STL; visual mesh filename=../meshes/link6.STL
- link link7: geometry collision mesh filename=../meshes/link7.STL; visual mesh filename=../meshes/link7.STL
- link link8: geometry collision mesh filename=../meshes/link8.STL; visual mesh filename=../meshes/link8.STL
